File: 48to7VConverter_Variable.kicad_pcb (KiCad board)
At the start: 2 copper layers, 74.3 x 40.9 mm, 17 parts, among them J1 XT_60_In, J2 XT_30_out, SW1 SW_DIP_x03, U1 TPS54360BDDAR

Commit message: Add files via upload
Parts:
- removed SW1: SW_DIP_x03, Button_Switch_THT:SW_DIP_SPSTx03_Slide_6.7x9.18mm_W7.62mm_P2.54mm_LowProfile
- added J3: XT_30_out, Connector_AMASS:AMASS_XT30UPB-M_1x02_P5.0mm_Vertical, F.Cu at (123.1, 97.0)
- J1: moved to B.Cu
- J2: value XT_30_out -> Conn_02x03_Odd_Even; footprint Connector_AMASS:AMASS_XT30UPB-M_1x02_P5.0mm_Vertical -> Connector_PinHeader_2.54mm:PinHeader_2x03_P2.54mm_Vertical
- moved J2 41.1 mm to (86.5, 117.5), turned to 0 degrees
Connections:
- J2 pad 1: /Vout -> Net-(J2-Pin_1)
- J2 pad 2: GND -> /Feedback
- R3 pad 2: Net-(R3-Pad2) -> Net-(J2-Pin_5)
- R4 pad 2: Net-(R4-Pad2) -> Net-(J2-Pin_3)
- R6 pad 2: Net-(R6-Pad2) -> Net-(J2-Pin_1)
- U1 pad EPAD: (no net) -> GND
Routing:
- net /Feedback: track 23.3 -> 37.6 mm
- net Net-(J2-Pin_1): track 0.00 -> 6.51 mm
- net Net-(J2-Pin_5): track 0.00 -> 6.46 mm
- net Net-(R3-Pad2): track 6.11 -> 0.00 mm
- net Net-(J2-Pin_3): track 0.00 -> 5.24 mm
- net Net-(R6-Pad2): track 5.00 -> 0.00 mm
- net Net-(R4-Pad2): track 4.52 -> 0.00 mm
- net GND: track 3.72 -> 7.57 mm, vias 1 -> 2
- net (no net): track 3.85 -> 0.00 mm, vias 1 -> 0
- net /Vout: track 103.3 -> 104.3 mm
- net Net-(D1-K): track 21.6 -> 20.7 mm
