File: 48to7VConverter_Variable.kicad_sch (KiCad schematic)
At the start: 17 parts, among them J1 XT_60_In, J2 XT_30_out, SW1 SW_DIP_x03, U1 TPS54360BDDAR

Commit message: Add files via upload
Parts:
- J2: renamed from SW1; value SW_DIP_x03 -> Conn_02x03_Odd_Even; footprint Button_Switch_THT:SW_DIP_SPSTx03_Slide_6.7x9.18mm_W7.62mm_P2.54mm_LowProfile -> Connector_PinHeader_2.54mm:PinHeader_2x03_P2.54mm_Vertical; symbol Switch:SW_DIP_x03 -> Connector_Generic:Conn_02x03_Odd_Even
- renumbered J2 to J3
Connections:
- net Feedback: now also J2.2 (Pin_2); no longer J2.5
- net at R4.2: now also J2.3 (Pin_3); no longer J2.2
- net at R3.2: now also J2.5 (Pin_5); no longer J2.3
Changed lines of the file:
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@@
-    (stroke (width 0) (type default))
-  )
-  (wire (pts (xy 177.8 118.11) (xy 177.8 120.65))
     (stroke (width 0) (type default))
   )
@@
     (stroke (width 0) (type default))
   )
-  (wire (pts (xy 181.61 118.11) (xy 181.61 120.65))
+  (wire (pts (xy 181.61 116.84) (xy 181.61 120.65))
     (stroke (width 0) (type default))
   )
@@
     (stroke (width 0) (type default))
   )
+  (wire (pts (xy 177.8 120.65) (xy 181.61 120.65))
+    (stroke (width 0) (type default))
+  )
   (wire (pts (xy 182.88 97.79) (xy 182.88 102.87))
     (stroke (width 0) (type default))
@@
     (stroke (width 0) (type default))
   )
+  (wire (pts (xy 180.34 116.84) (xy 181.61 116.84))
+    (stroke (width 0) (type default))
+  )
   (wire (pts (xy 181.61 81.28) (xy 193.04 81.28))
     (stroke (width 0) (type default))
@@
     (stroke (width 0) (type default))
   )
+  (wire (pts (xy 177.8 115.57) (xy 177.8 120.65))
+    (stroke (width 0) (type default))
+  )
   (wire (pts (xy 132.08 83.82) (xy 132.08 81.28))
     (stroke (width 0) (type default))
@@
     (stroke (width 0) (type default))
   )
-  (wire (pts (xy 182.88 118.11) (xy 182.88 120.65))
+  (wire (pts (xy 182.88 115.57) (xy 182.88 120.65))
     (stroke (width 0) (type default))
   )
@@
     (stroke (width 0) (type default))
   )
-  (wire (pts (xy 180.34 118.11) (xy 181.61 118.11))
-    (stroke (width 0) (type default))
-  )
   (wire (pts (xy 168.91 92.71) (xy 168.91 101.6))
     (stroke (width 0) (type default))
@@
     (stroke (width 0) (type default))
   )
+  (wire (pts (xy 180.34 115.57) (xy 180.34 116.84))
+    (stroke (width 0) (type default))
+  )
   (wire (pts (xy 125.73 96.52) (xy 125.73 99.06))
     (stroke (width 0) (type default))
@@
   )
   (wire (pts (xy 125.73 106.68) (xy 125.73 107.95))
-    (stroke (width 0) (type default))
-  )
-  (wire (pts (xy 177.8 120.65) (xy 181.61 120.65))
     (stroke (width 0) (type default))
   )
@@
   (symbol (lib_id "Connector:Conn_01x02_Pin") (at 248.92 88.9 0) (unit 1)
     (in_bom yes) (on_board yes) (dnp no)
-    (property "Reference" "J2" (at 249.555 85.09 0)
+    (property "Reference" "J3" (at 249.555 85.09 0)
       (effects (font (size 1.27 1.27)))
     )
@@
       (project "48to7VConverter_Variable"
         (path "/7725f0b8-cb64-45b3-baea-c04ebf2b9791"
-          (reference "J2") (unit 1)
+          (reference "J3") (unit 1)
         )
       )
@@
   (symbol (lib_id "Connector:Conn_01x02_Pin") (at 29.21 78.74 0) (unit 1)
     (in_bom yes) (on_board yes) (dnp no)
-    (property "Reference" "J1" (at 29.845 74.295 0)
+    (property "Reference" "J1" (at 26.67 80.01 0)
       (effects (font (size 1.27 1.27)))
     )
@@
     )
   )
-  (symbol (lib_id "Switch:SW_DIP_x03") (at 177.8 110.49 270) (unit 1)
-    (in_bom yes) (on_board yes) (dnp no) (fields_autoplaced)
-    (property "Reference" "SW1" (at 186.69 109.855 90)
-      (effects (font (size 1.27 1.27)) (justify left))
-    )
-    (property "Value" "SW_DIP_x03" (at 186.69 112.395 90)
-      (effects (font (size 1.27 1.27)) (justify left))
-    )
-    (property "Footprint" "Button_Switch_THT:SW_DIP_SPSTx03_Slide_6.7x9.18mm_W7.62mm_P2.54mm_LowProfile" (at 177.8 110.49 0)
-      (effects (font (size 1.27 1.27)) hide)
-    )
-    (property "Datasheet" "~" (at 177.8 110.49 0)
+  (symbol (lib_id "Connector_Generic:Conn_02x03_Odd_Even") (at 180.34 107.95 270) (unit 1)
+    (in_bom yes) (on_board yes) (dnp no)
+    (property "Reference" "J2" (at 186.69 109.22 90)
+      (effects (font (size 1.27 1.27)))
+    )
+    (property "Value" "Conn_02x03_Odd_Even" (at 195.58 113.03 90)
+      (effects (font (size 1.27 1.27)))
+    )
+    (property "Footprint" "Connector_PinHeader_2.54mm:PinHeader_2x03_P2.54mm_Vertical" (at 180.34 107.95 0)
+      (effects (font (size 1.27 1.27)) hide)
+    )
+    (property "Datasheet" "~" (at 180.34 107.95 0)
       (effects (font (size 1.27 1.27)) hide)
     )
@@
       (project "48to7VConverter_Variable"
         (path "/7725f0b8-cb64-45b3-baea-c04ebf2b9791"
-          (reference "SW1") (unit 1)
-        )
-      )
+          (reference "J2") (unit 1)
+        )
+      )
